Commit message: Stabilize G1 omniwheel contacts for Newton

File: urdf/galbot_one_golf.urdf (robot description, URDF)
Before this commit: robot galbot_one_golf, 104 links, 103 joints
Links:
- link wheel_1_passive_0: geometry collision cylinder length=0.065 radius=0.025
- link wheel_1_passive_1: geometry collision cylinder length=0.065 radius=0.025
- link wheel_1_passive_2: geometry collision cylinder length=0.065 radius=0.025
- link wheel_1_passive_3: geometry collision cylinder length=0.065 radius=0.025
- link wheel_1_passive_4: geometry collision cylinder length=0.065 radius=0.025
- link wheel_1_passive_5: geometry collision cylinder length=0.065 radius=0.025
- link wheel_1_passive_6: geometry collision cylinder length=0.065 radius=0.025
- link wheel_1_passive_7: geometry collision cylinder length=0.065 radius=0.025
- link wheel_1_passive_8: geometry collision cylinder length=0.065 radius=0.025
- link wheel_1_passive_9: geometry collision cylinder length=0.065 radius=0.025
- link wheel_2_passive_0: geometry collision cylinder length=0.065 radius=0.025
- link wheel_2_passive_1: geometry collision cylinder length=0.065 radius=0.025
- link wheel_2_passive_2: geometry collision cylinder length=0.065 radius=0.025
- link wheel_2_passive_3: geometry collision cylinder length=0.065 radius=0.025
- link wheel_2_passive_4: geometry collision cylinder length=0.065 radius=0.025
- link wheel_2_passive_5: geometry collision cylinder length=0.065 radius=0.025
- link wheel_2_passive_6: geometry collision cylinder length=0.065 radius=0.025
- link wheel_2_passive_7: geometry collision cylinder length=0.065 radius=0.025
- link wheel_2_passive_8: geometry collision cylinder length=0.065 radius=0.025
- link wheel_2_passive_9: geometry collision cylinder length=0.065 radius=0.025
- link wheel_3_passive_0: geometry collision cylinder length=0.065 radius=0.025
- link wheel_3_passive_1: geometry collision cylinder length=0.065 radius=0.025
- link wheel_3_passive_2: geometry collision cylinder length=0.065 radius=0.025
- link wheel_3_passive_3: geometry collision cylinder length=0.065 radius=0.025
- link wheel_3_passive_4: geometry collision cylinder length=0.065 radius=0.025
- link wheel_3_passive_5: geometry collision cylinder length=0.065 radius=0.025
- link wheel_3_passive_6: geometry collision cylinder length=0.065 radius=0.025
- link wheel_3_passive_7: geometry collision cylinder length=0.065 radius=0.025
- link wheel_3_passive_8: geometry collision cylinder length=0.065 radius=0.025
- link wheel_3_passive_9: geometry collision cylinder length=0.065 radius=0.025
- link wheel_4_passive_0: geometry collision cylinder length=0.065 radius=0.025
- link wheel_4_passive_1: geometry collision cylinder length=0.065 radius=0.025
- link wheel_4_passive_2: geometry collision cylinder length=0.065 radius=0.025
- link wheel_4_passive_3: geometry collision cylinder length=0.065 radius=0.025
- link wheel_4_passive_4: geometry collision cylinder length=0.065 radius=0.025
- link wheel_4_passive_5: geometry collision cylinder length=0.065 radius=0.025
- link wheel_4_passive_6: geometry collision cylinder length=0.065 radius=0.025
- link wheel_4_passive_7: geometry collision cylinder length=0.065 radius=0.025
- link wheel_4_passive_8: geometry collision cylinder length=0.065 radius=0.025
- link wheel_4_passive_9: geometry collision cylinder length=0.065 radius=0.025
Joints:
- joint wheel_1_passive_0_joint: origin xyz=0 0.025 0.0 rpy=0.0 0 0 -> xyz=0 0.08 0.0 rpy=0.0 0 0
- joint wheel_1_passive_1_joint: origin xyz=0 0.02022542485937369 0.014694631307311828 rpy=0.6283185307179586 0 0 -> xyz=0 0.06472135954999579 0.04702282018339785 rpy=0.6283185307179586 0 0
- joint wheel_1_passive_2_joint: origin xyz=0 0.007725424859373687 0.02377641290737884 rpy=1.2566370614359172 0 0 -> xyz=0 0.024721359549995797 0.07608452130361229 rpy=1.2566370614359172 0 0
- joint wheel_1_passive_3_joint: origin xyz=0 -0.007725424859373684 0.023776412907378842 rpy=1.8849555921538759 0 0 -> xyz=0 -0.024721359549995787 0.07608452130361229 rpy=1.8849555921538759 0 0
- joint wheel_1_passive_4_joint: origin xyz=0 -0.020225424859373686 0.014694631307311832 rpy=2.5132741228718345 0 0 -> xyz=0 -0.06472135954999579 0.04702282018339786 rpy=2.5132741228718345 0 0
- joint wheel_1_passive_5_joint: origin xyz=0 -0.025 3.061616997868383e-18 rpy=3.141592653589793 0 0 -> xyz=0 -0.08 9.797174393178826e-18 rpy=3.141592653589793 0 0
- joint wheel_1_passive_6_joint: origin xyz=0 -0.02022542485937369 -0.014694631307311827 rpy=3.7699111843077517 0 0 -> xyz=0 -0.0647213595499958 -0.047022820183397845 rpy=3.7699111843077517 0 0
- joint wheel_1_passive_7_joint: origin xyz=0 -0.007725424859373689 -0.02377641290737884 rpy=4.39822971502571 0 0 -> xyz=0 -0.024721359549995804 -0.07608452130361229 rpy=4.39822971502571 0 0
- joint wheel_1_passive_8_joint: origin xyz=0 0.007725424859373681 -0.023776412907378842 rpy=5.026548245743669 0 0 -> xyz=0 0.02472135954999578 -0.07608452130361229 rpy=5.026548245743669 0 0
- joint wheel_1_passive_9_joint: origin xyz=0 0.020225424859373686 -0.014694631307311835 rpy=5.654866776461628 0 0 -> xyz=0 0.06472135954999579 -0.04702282018339787 rpy=5.654866776461628 0 0
- joint wheel_2_passive_0_joint: origin xyz=0 0.025 0.0 rpy=0.0 0 0 -> xyz=0 0.08 0.0 rpy=0.0 0 0
- joint wheel_2_passive_1_joint: origin xyz=0 0.02022542485937369 0.014694631307311828 rpy=0.6283185307179586 0 0 -> xyz=0 0.06472135954999579 0.04702282018339785 rpy=0.6283185307179586 0 0
- joint wheel_2_passive_2_joint: origin xyz=0 0.007725424859373687 0.02377641290737884 rpy=1.2566370614359172 0 0 -> xyz=0 0.024721359549995797 0.07608452130361229 rpy=1.2566370614359172 0 0
- joint wheel_2_passive_3_joint: origin xyz=0 -0.007725424859373684 0.023776412907378842 rpy=1.8849555921538759 0 0 -> xyz=0 -0.024721359549995787 0.07608452130361229 rpy=1.8849555921538759 0 0
- joint wheel_2_passive_4_joint: origin xyz=0 -0.020225424859373686 0.014694631307311832 rpy=2.5132741228718345 0 0 -> xyz=0 -0.06472135954999579 0.04702282018339786 rpy=2.5132741228718345 0 0
- joint wheel_2_passive_5_joint: origin xyz=0 -0.025 3.061616997868383e-18 rpy=3.141592653589793 0 0 -> xyz=0 -0.08 9.797174393178826e-18 rpy=3.141592653589793 0 0
- joint wheel_2_passive_6_joint: origin xyz=0 -0.02022542485937369 -0.014694631307311827 rpy=3.7699111843077517 0 0 -> xyz=0 -0.0647213595499958 -0.047022820183397845 rpy=3.7699111843077517 0 0
- joint wheel_2_passive_7_joint: origin xyz=0 -0.007725424859373689 -0.02377641290737884 rpy=4.39822971502571 0 0 -> xyz=0 -0.024721359549995804 -0.07608452130361229 rpy=4.39822971502571 0 0
- joint wheel_2_passive_8_joint: origin xyz=0 0.007725424859373681 -0.023776412907378842 rpy=5.026548245743669 0 0 -> xyz=0 0.02472135954999578 -0.07608452130361229 rpy=5.026548245743669 0 0
- joint wheel_2_passive_9_joint: origin xyz=0 0.020225424859373686 -0.014694631307311835 rpy=5.654866776461628 0 0 -> xyz=0 0.06472135954999579 -0.04702282018339787 rpy=5.654866776461628 0 0
- joint wheel_3_passive_0_joint: origin xyz=0 0.025 0.0 rpy=0.0 0 0 -> xyz=0 0.08 0.0 rpy=0.0 0 0
- joint wheel_3_passive_1_joint: origin xyz=0 0.02022542485937369 0.014694631307311828 rpy=0.6283185307179586 0 0 -> xyz=0 0.06472135954999579 0.04702282018339785 rpy=0.6283185307179586 0 0
- joint wheel_3_passive_2_joint: origin xyz=0 0.007725424859373687 0.02377641290737884 rpy=1.2566370614359172 0 0 -> xyz=0 0.024721359549995797 0.07608452130361229 rpy=1.2566370614359172 0 0
- joint wheel_3_passive_3_joint: origin xyz=0 -0.007725424859373684 0.023776412907378842 rpy=1.8849555921538759 0 0 -> xyz=0 -0.024721359549995787 0.07608452130361229 rpy=1.8849555921538759 0 0
- joint wheel_3_passive_4_joint: origin xyz=0 -0.020225424859373686 0.014694631307311832 rpy=2.5132741228718345 0 0 -> xyz=0 -0.06472135954999579 0.04702282018339786 rpy=2.5132741228718345 0 0
- joint wheel_3_passive_5_joint: origin xyz=0 -0.025 3.061616997868383e-18 rpy=3.141592653589793 0 0 -> xyz=0 -0.08 9.797174393178826e-18 rpy=3.141592653589793 0 0
- joint wheel_3_passive_6_joint: origin xyz=0 -0.02022542485937369 -0.014694631307311827 rpy=3.7699111843077517 0 0 -> xyz=0 -0.0647213595499958 -0.047022820183397845 rpy=3.7699111843077517 0 0
- joint wheel_3_passive_7_joint: origin xyz=0 -0.007725424859373689 -0.02377641290737884 rpy=4.39822971502571 0 0 -> xyz=0 -0.024721359549995804 -0.07608452130361229 rpy=4.39822971502571 0 0
- joint wheel_3_passive_8_joint: origin xyz=0 0.007725424859373681 -0.023776412907378842 rpy=5.026548245743669 0 0 -> xyz=0 0.02472135954999578 -0.07608452130361229 rpy=5.026548245743669 0 0
- joint wheel_3_passive_9_joint: origin xyz=0 0.020225424859373686 -0.014694631307311835 rpy=5.654866776461628 0 0 -> xyz=0 0.06472135954999579 -0.04702282018339787 rpy=5.654866776461628 0 0
- joint wheel_4_passive_0_joint: origin xyz=0 0.025 0.0 rpy=0.0 0 0 -> xyz=0 0.08 0.0 rpy=0.0 0 0
- joint wheel_4_passive_1_joint: origin xyz=0 0.02022542485937369 0.014694631307311828 rpy=0.6283185307179586 0 0 -> xyz=0 0.06472135954999579 0.04702282018339785 rpy=0.6283185307179586 0 0
- joint wheel_4_passive_2_joint: origin xyz=0 0.007725424859373687 0.02377641290737884 rpy=1.2566370614359172 0 0 -> xyz=0 0.024721359549995797 0.07608452130361229 rpy=1.2566370614359172 0 0
- joint wheel_4_passive_3_joint: origin xyz=0 -0.007725424859373684 0.023776412907378842 rpy=1.8849555921538759 0 0 -> xyz=0 -0.024721359549995787 0.07608452130361229 rpy=1.8849555921538759 0 0
- joint wheel_4_passive_4_joint: origin xyz=0 -0.020225424859373686 0.014694631307311832 rpy=2.5132741228718345 0 0 -> xyz=0 -0.06472135954999579 0.04702282018339786 rpy=2.5132741228718345 0 0
- joint wheel_4_passive_5_joint: origin xyz=0 -0.025 3.061616997868383e-18 rpy=3.141592653589793 0 0 -> xyz=0 -0.08 9.797174393178826e-18 rpy=3.141592653589793 0 0
- joint wheel_4_passive_6_joint: origin xyz=0 -0.02022542485937369 -0.014694631307311827 rpy=3.7699111843077517 0 0 -> xyz=0 -0.0647213595499958 -0.047022820183397845 rpy=3.7699111843077517 0 0
- joint wheel_4_passive_7_joint: origin xyz=0 -0.007725424859373689 -0.02377641290737884 rpy=4.39822971502571 0 0 -> xyz=0 -0.024721359549995804 -0.07608452130361229 rpy=4.39822971502571 0 0
- joint wheel_4_passive_8_joint: origin xyz=0 0.007725424859373681 -0.023776412907378842 rpy=5.026548245743669 0 0 -> xyz=0 0.02472135954999578 -0.07608452130361229 rpy=5.026548245743669 0 0
- joint wheel_4_passive_9_joint: origin xyz=0 0.020225424859373686 -0.014694631307311835 rpy=5.654866776461628 0 0 -> xyz=0 0.06472135954999579 -0.04702282018339787 rpy=5.654866776461628 0 0

File: urdf/galbot_one_golf_fixed_base.urdf (robot description, URDF)
Before this commit: robot galbot_one_golf, 64 links, 63 joints
Links:
- link wheel_1: geometry collision cylinder length=0.065 radius=0.025; collision cylinder length=0.065 radius=0.025
- link wheel_2: geometry collision cylinder length=0.065 radius=0.025; collision cylinder length=0.065 radius=0.025
- link wheel_3: geometry collision cylinder length=0.065 radius=0.025; collision cylinder length=0.065 radius=0.025
- link wheel_4: geometry collision cylinder length=0.065 radius=0.025; collision cylinder length=0.065 radius=0.025

File: xacro/components/omniwheel_10.xacro (robot description, xacro)
@@ -5,6 +5,8 @@
   <xacro:arg name="enable_passive_wheels" default="false"/>
   <xacro:property name="PI" value="3.1415926535897931"/>
-  <!-- 被动轮宏定义 -->
-  <xacro:macro name="passive_wheel" params="parent_link passive_wheel_name radius angle sphere_radius:='0.08'">
+  <!-- URDF has no capsule primitive.  Author the same total roller length as a
+       cylinder here; scripts/finalize_mjcf.py converts it to the rounded MJCF
+       capsule used by Newton without changing its local-Z hinge axis. -->
+  <xacro:macro name="passive_wheel" params="parent_link passive_wheel_name center_radius angle collision_radius collision_half_length">
     <!-- 被动轮链接 -->
     <link name="${passive_wheel_name}">
@@ -16,5 +18,7 @@
       <collision>
         <geometry>
-          <sphere radius="${float(sphere_radius)}"/>
+          <cylinder
+            radius="${float(collision_radius)}"
+            length="${2.0 * (float(collision_radius) + float(collision_half_length))}"/>
         </geometry>
       </collision>
@@ -23,5 +27,5 @@
     <joint name="${passive_wheel_name}_joint" type="continuous">
       <!-- 让y轴负方向指向圆心：被动轮在角度angle位置，需要绕x轴旋转angle角度使y轴负方向指向圆心 -->
-      <origin xyz="0 ${float(radius) * cos(float(angle))} ${float(radius) * sin(float(angle))}" rpy="${float(angle)} 0 0"/>
+      <origin xyz="0 ${float(center_radius) * cos(float(angle))} ${float(center_radius) * sin(float(angle))}" rpy="${float(angle)} 0 0"/>
       <parent link="${parent_link}"/>
       <child link="${passive_wheel_name}"/>
@@ -30,5 +34,5 @@
   </xacro:macro>
   <!-- 递归宏：创建被动轮循环 -->
-  <xacro:macro name="create_passive_wheels" params="parent_link wheel_name indices:=^ angle_step passive_wheel_radius_actual">
+  <xacro:macro name="create_passive_wheels" params="parent_link wheel_name indices:=^ angle_step roller_center_radius roller_collision_radius roller_collision_half_length">
     <xacro:if value="${indices}">
       <!-- 弹出第一个索引 -->
@@ -40,6 +44,8 @@
         parent_link="${parent_link}"
         passive_wheel_name="${wheel_name}_passive_${index}"
-        radius="${passive_wheel_radius_actual}"
-        angle="${angle}"/>
+        center_radius="${roller_center_radius}"
+        angle="${angle}"
+        collision_radius="${roller_collision_radius}"
+        collision_half_length="${roller_collision_half_length}"/>
       <!-- 递归调用自己 -->
       <xacro:create_passive_wheels
@@ -48,31 +54,39 @@
         indices="${indices}"
         angle_step="${angle_step}"
-        passive_wheel_radius_actual="${passive_wheel_radius_actual}"/>
+        roller_center_radius="${roller_center_radius}"
+        roller_collision_radius="${roller_collision_radius}"
+        roller_collision_half_length="${roller_collision_half_length}"/>
     </xacro:if>
   </xacro:macro>
-  <xacro:macro name="wheel_collision_sphere" params="wheel_name index radius angle sphere_radius">
+  <xacro:macro name="wheel_collision_cylinder" params="wheel_name index center_radius angle collision_radius collision_half_length">
     <collision name="${wheel_name}_collision_${index}">
-      <origin xyz="0 ${float(radius) * cos(float(angle))} ${float(radius) * sin(float(angle))}"/>
+      <origin
+        xyz="0 ${float(center_radius) * cos(float(angle))} ${float(center_radius) * sin(float(angle))}"
+        rpy="${float(angle)} 0 0"/>
       <geometry>
-        <sphere radius="${float(sphere_radius)}"/>
+        <cylinder
+          radius="${float(collision_radius)}"
+          length="${2.0 * (float(collision_radius) + float(collision_half_length))}"/>
       </geometry>
     </collision>
   </xacro:macro>
-  <xacro:macro name="create_wheel_collision_spheres" params="wheel_name indices:=^ angle_step radius sphere_radius">
+  <xacro:macro name="create_wheel_collision_cylinders" params="wheel_name indices:=^ angle_step roller_center_radius roller_collision_radius roller_collision_half_length">
     <xacro:if value="${indices}">
       <xacro:property name="index" value="${indices.pop(0)}"/>
       <xacro:property name="angle" value="${float(index) * float(angle_step)}"/>
-      <xacro:wheel_collision_sphere
+      <xacro:wheel_collision_cylinder
         wheel_name="${wheel_name}"
         index="${index}"
-        radius="${radius}"
+        center_radius="${roller_center_radius}"
         angle="${angle}"
-        sphere_radius="${sphere_radius}"/>
-      <xacro:create_wheel_collision_spheres
+        collision_radius="${roller_collision_radius}"
+        collision_half_length="${roller_collision_half_length}"/>
+      <xacro:create_wheel_collision_cylinders
         wheel_name="${wheel_name}"
         indices="${indices}"
         angle_step="${angle_step}"
-        radius="${radius}"
-        sphere_radius="${sphere_radius}"/>
+        roller_center_radius="${roller_center_radius}"
+        roller_collision_radius="${roller_collision_radius}"
+        roller_collision_half_length="${roller_collision_half_length}"/>
     </xacro:if>
   </xacro:macro>
@@ -81,6 +95,6 @@
                 inertial_origin_xyz:='0.0026089441594678298 -1.3189703553351252e-07 2.8695680726054107e-07'
                 ixx:='0.012235' ixy:='-0.0' ixz:='0.0' iyy:='0.006629' iyz:='0.0' izz:='0.006629'
-                passive_wheel_radius:='0.02' wheel_radius:='0.15' num_passive_wheels:='10'
-                wheel_collision_radius:='0.025' wheel_collision_sphere_radius:='0.08'
+                num_passive_wheels:='10'
+                roller_center_radius:='0.08' roller_collision_radius:='0.025' roller_collision_half_length:='0.0075'
                 enable_passive_wheels:='false'">
     <!-- 轮子链接 -->
@@ -98,10 +112,11 @@
       <xacro:unless value="${enable_passive_wheels}">
         <xacro:property name="wheel_collision_indices" value="${[0,1,2,3,4,5,6,7,8,9]}"/>
-        <xacro:create_wheel_collision_spheres
+        <xacro:create_wheel_collision_cylinders
           wheel_name="${wheel_name}"
           indices="${list(wheel_collision_indices)}"
           angle_step="${2*PI / float(num_passive_wheels)}"
-          radius="${wheel_collision_radius}"
-          sphere_radius="${wheel_collision_sphere_radius}"/>
+          roller_center_radius="${roller_center_radius}"
+          roller_collision_radius="${roller_collision_radius}"
+          roller_collision_half_length="${roller_collision_half_length}"/>
       </xacro:unless>
     </link>
@@ -111,5 +126,4 @@
       <xacro:property name="num_passive_wheels_float" value="${float(num_passive_wheels)}"/>
       <xacro:property name="angle_step" value="${2*PI / num_passive_wheels_float}"/>
-      <xacro:property name="passive_wheel_radius_actual" value="0.025"/>
       <xacro:property name="indices" value="${[0,1,2,3,4,5,6,7,8,9]}"/>
       <xacro:create_passive_wheels
@@ -118,5 +132,7 @@
         indices="${list(indices)}"
         angle_step="${angle_step}"
-        passive_wheel_radius_actual="${passive_wheel_radius_actual}"/>
+        roller_center_radius="${roller_center_radius}"
+        roller_collision_radius="${roller_collision_radius}"
+        roller_collision_half_length="${roller_collision_half_length}"/>
     </xacro:if>
   </xacro:macro>

Commit message: Use base_link as the robot root

File: urdf/galbot_one_golf.urdf (robot description, URDF)
Before this commit: robot galbot_one_golf, 104 links, 103 joints
Joints:
- joint base_footprint_joint: child base_link -> base_footprint; origin xyz=0 0 0.028166 -> xyz=0 0 -0.028166; parent base_footprint -> base_link

File: urdf/galbot_one_golf_fixed_base.urdf (robot description, URDF)
Before this commit: robot galbot_one_golf, 64 links, 63 joints
Joints:
- joint base_footprint_joint: child base_link -> base_footprint; origin xyz=0 0 0.028166 -> xyz=0 0 -0.028166; parent base_footprint -> base_link

File: xacro/components/omni_chassis.xacro (robot description, xacro)
@@ -8,11 +8,11 @@
   <xacro:macro name="GalbotChassisV2" params="enable_wheel_joints:='false' enable_passive_wheels:='false'">
     <!-- Robot Base Link -->
+    <link name="base_link"/>
     <link name="base_footprint"/>
     <joint name="base_footprint_joint" type="fixed">
-      <origin xyz="0 0 0.028166"/>
-      <parent link="base_footprint"/>
-      <child link="base_link"/>
+      <origin xyz="0 0 -0.028166"/>
+      <parent link="base_link"/>
+      <child link="base_footprint"/>
     </joint>
-    <link name="base_link"/>
     <joint name="omni_chassis_joint" type="fixed">
       <parent link="base_link"/>
