Commit message: Fix omni-wheel mass accounting

File: urdf/galbot_one_golf.urdf (robot description, URDF)
Before this commit: robot galbot_one_golf, 104 links, 103 joints
Links:
- link omni_chassis_base_link: mass 30.15 -> 22.926
- link wheel_1: mass 4.24803000494366 -> 1.306
- link wheel_1_passive_0: mass 0.1 -> 0.05
- link wheel_1_passive_1: mass 0.1 -> 0.05
- link wheel_1_passive_2: mass 0.1 -> 0.05
- link wheel_1_passive_3: mass 0.1 -> 0.05
- link wheel_1_passive_4: mass 0.1 -> 0.05
- link wheel_1_passive_5: mass 0.1 -> 0.05
- link wheel_1_passive_6: mass 0.1 -> 0.05
- link wheel_1_passive_7: mass 0.1 -> 0.05
- link wheel_1_passive_8: mass 0.1 -> 0.05
- link wheel_1_passive_9: mass 0.1 -> 0.05
- link wheel_2: mass 4.24803000494366 -> 1.306
- link wheel_2_passive_0: mass 0.1 -> 0.05
- link wheel_2_passive_1: mass 0.1 -> 0.05
- link wheel_2_passive_2: mass 0.1 -> 0.05
- link wheel_2_passive_3: mass 0.1 -> 0.05
- link wheel_2_passive_4: mass 0.1 -> 0.05
- link wheel_2_passive_5: mass 0.1 -> 0.05
- link wheel_2_passive_6: mass 0.1 -> 0.05
- link wheel_2_passive_7: mass 0.1 -> 0.05
- link wheel_2_passive_8: mass 0.1 -> 0.05
- link wheel_2_passive_9: mass 0.1 -> 0.05
- link wheel_3: mass 4.24803000494366 -> 1.306
- link wheel_3_passive_0: mass 0.1 -> 0.05
- link wheel_3_passive_1: mass 0.1 -> 0.05
- link wheel_3_passive_2: mass 0.1 -> 0.05
- link wheel_3_passive_3: mass 0.1 -> 0.05
- link wheel_3_passive_4: mass 0.1 -> 0.05
- link wheel_3_passive_5: mass 0.1 -> 0.05
- link wheel_3_passive_6: mass 0.1 -> 0.05
- link wheel_3_passive_7: mass 0.1 -> 0.05
- link wheel_3_passive_8: mass 0.1 -> 0.05
- link wheel_3_passive_9: mass 0.1 -> 0.05
- link wheel_4: mass 4.24803000494366 -> 1.306
- link wheel_4_passive_0: mass 0.1 -> 0.05
- link wheel_4_passive_1: mass 0.1 -> 0.05
- link wheel_4_passive_2: mass 0.1 -> 0.05
- link wheel_4_passive_3: mass 0.1 -> 0.05
- link wheel_4_passive_4: mass 0.1 -> 0.05
- link wheel_4_passive_5: mass 0.1 -> 0.05
- link wheel_4_passive_6: mass 0.1 -> 0.05
- link wheel_4_passive_7: mass 0.1 -> 0.05
- link wheel_4_passive_8: mass 0.1 -> 0.05
- link wheel_4_passive_9: mass 0.1 -> 0.05

File: urdf/galbot_one_golf_fixed_base.urdf (robot description, URDF)
Before this commit: robot galbot_one_golf, 64 links, 63 joints
Links:
- link omni_chassis_base_link: mass 30.15 -> 22.926
- link wheel_1: mass 4.24803000494366 -> 1.806
- link wheel_2: mass 4.24803000494366 -> 1.806
- link wheel_3: mass 4.24803000494366 -> 1.806
- link wheel_4: mass 4.24803000494366 -> 1.806

File: xacro/components/omni_chassis.xacro (robot description, xacro)
@@ -6,4 +6,7 @@
   <xacro:property name="PI" value="3.1415926535897931"/>
   <xacro:include filename="omniwheel_10.xacro"/>
+  <!-- The measured 30.15 kg chassis module includes four complete wheel assemblies. -->
+  <xacro:property name="omni_chassis_module_mass" value="30.15"/>
+  <xacro:property name="omni_chassis_wheel_count" value="4"/>
   <xacro:macro name="GalbotChassisV2" params="enable_wheel_joints:='false' enable_passive_wheels:='false'">
     <!-- Robot Base Link -->
@@ -21,7 +24,8 @@
     <link name="omni_chassis_base_link">
       <inertial>
-        <origin xyz="0.02079 0.00615 0.07261"/>
-        <mass value="30.15"/>
-        <inertia ixx="0.3317069394" ixy="3.760583e-05" ixz="3.706221e-05" iyy="0.32081635568" iyz="1.303674e-05" izz="0.55833152838"/>
+        <!-- Motors and chassis brackets stay here; rotating outputs live on the wheel links. -->
+        <origin xyz="0.027340944778854 0.008087869667626 0.072854427768648"/>
+        <mass value="${float(omni_chassis_module_mass) - float(omni_chassis_wheel_count) * float(omniwheel_output_mass)}"/>
+        <inertia ixx="0.09495588499632361" ixy="0.001252298388256994" ixz="0.0001902740573022943" iyy="0.08031837253490508" iyz="0.00005835914793213606" izz="0.1019001895297286"/>
       </inertial>
       <visual>

File: xacro/components/omniwheel_10.xacro (robot description, xacro)
@@ -5,4 +5,7 @@
   <xacro:arg name="enable_passive_wheels" default="false"/>
   <xacro:property name="PI" value="3.1415926535897931"/>
+  <!-- Measured rotating output assembly: 2.268 - 0.380 - 0.082 kg. -->
+  <xacro:property name="omniwheel_output_mass" value="1.806"/>
+  <xacro:property name="omniwheel_passive_roller_mass" value="0.05"/>
   <!-- 被动轮宏定义 -->
   <xacro:macro name="passive_wheel" params="parent_link passive_wheel_name radius angle sphere_radius:='0.08'">
@@ -11,6 +14,6 @@
       <inertial>
         <origin xyz="0 0 0"/>
-        <mass value="0.1"/>
-        <inertia ixx="0.0001" ixy="0.0" ixz="0.0" iyy="0.0001" iyz="0.0" izz="0.0001"/>
+        <mass value="${omniwheel_passive_roller_mass}"/>
+        <inertia ixx="0.00004" ixy="0.0" ixz="0.0" iyy="0.00004" iyz="0.0" izz="0.00004"/>
       </inertial>
       <collision>
@@ -80,5 +83,5 @@
   <xacro:macro name="wheel" params="wheel_name
                 inertial_origin_xyz:='0.0026089441594678298 -1.3189703553351252e-07 2.8695680726054107e-07'
-                ixx:='0.012235' ixy:='-0.0' ixz:='0.0' iyy:='0.006629' iyz:='0.0' izz:='0.006629'
+                ixx:='0.005201566367065' ixy:='0.0' ixz:='0.0' iyy:='0.002818241393321' iyz:='0.0' izz:='0.002818241393321'
                 passive_wheel_radius:='0.02' wheel_radius:='0.15' num_passive_wheels:='10'
                 wheel_collision_radius:='0.025' wheel_collision_sphere_radius:='0.08'
@@ -87,7 +90,15 @@
     <link name="${wheel_name}">
       <inertial>
-        <origin xyz="${inertial_origin_xyz}"/>
-        <mass value="4.24803000494366"/>
-        <inertia ixx="${ixx}" ixy="${ixy}" ixz="${ixz}" iyy="${iyy}" iyz="${iyz}" izz="${izz}"/>
+        <xacro:if value="${enable_passive_wheels}">
+          <!-- The ten roller bodies own 0.5 kg of the 1.806 kg assembly. -->
+          <origin xyz="0.003607774235833767 -1.823936035019323e-07 3.968177595042398e-07"/>
+          <mass value="${float(omniwheel_output_mass) - float(num_passive_wheels) * float(omniwheel_passive_roller_mass)}"/>
+          <inertia ixx="0.004489066366996529" ixy="-2.379273632891010e-10" ixz="5.176376880170815e-10" iyy="0.002257285152503005" iyz="-2.616953691508134e-14" izz="0.002257285152547911"/>
+        </xacro:if>
+        <xacro:unless value="${enable_passive_wheels}">
+          <origin xyz="${inertial_origin_xyz}"/>
+          <mass value="${omniwheel_output_mass}"/>
+          <inertia ixx="${ixx}" ixy="${ixy}" ixz="${ixz}" iyy="${iyy}" iyz="${iyz}" izz="${izz}"/>
+        </xacro:unless>
       </inertial>
       <visual>

Commit message: Fix gripper TCP frame orientation

File: urdf/galbot_one_golf.urdf (robot description, URDF)
Before this commit: robot galbot_one_golf, 104 links, 103 joints
Joints:
- joint left_gripper_tcp_joint: origin xyz=0.13996 0 0 rpy=1.5707963267948966 0 0 -> xyz=0.13996 0 0 rpy=-1.5707963267948966 0 0
- joint right_gripper_tcp_joint: origin xyz=0.13996 0 0 rpy=1.5707963267948966 0 0 -> xyz=0.13996 0 0 rpy=-1.5707963267948966 0 0

File: urdf/galbot_one_golf_fixed_base.urdf (robot description, URDF)
Before this commit: robot galbot_one_golf, 64 links, 63 joints
Joints:
- joint left_gripper_tcp_joint: origin xyz=0.13996 0 0 rpy=1.5707963267948966 0 0 -> xyz=0.13996 0 0 rpy=-1.5707963267948966 0 0
- joint right_gripper_tcp_joint: origin xyz=0.13996 0 0 rpy=1.5707963267948966 0 0 -> xyz=0.13996 0 0 rpy=-1.5707963267948966 0 0

File: xacro/components/galbot_gripper.xacro (robot description, xacro)
@@ -365,5 +365,5 @@
 			<parent link="${prefix}gripper_base_link"/>
 			<child link="${prefix}gripper_tcp_link"/>
-			<origin rpy="1.5707963267948966 0 0" xyz="0.13996 0 0"/>
+			<origin rpy="-1.5707963267948966 0 0" xyz="0.13996 0 0"/>
 		</joint>
 	</xacro:macro>
